File: hardware/rpi-avionics/rpi-avionics.kicad_sch (KiCad schematic)
At the start: 17 parts, among them J1 To Controller, J2 Panel Data, J3 Panel Audio, J4 Audio from Panel, J5 Music to Panel, J6 Alert to Panel, J7 Thermal Cam, J8 Temp Sensor, P1 Raspberry_Pi_4, T1 Panel Left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

Commit message: panel and avionics boards
Parts:
- added C1, C2, C3, C4: 0.1µ, Capacitor_THT:C_Disc_D5.0mm_W2.5mm_P5.00mm, symbol Device:C
- added C5, C6: 1µF, Capacitor_THT:C_Disc_D5.0mm_W2.5mm_P5.00mm, symbol Device:C
- added J10: Fan, Connector_JST:JST_XH_B2B-XH-A_1x02_P2.50mm_Vertical, symbol Connector:Screw_Terminal_01x02
- added J12: Thermal 1, Connector_JST:JST_XH_B2B-XH-A_1x02_P2.50mm_Vertical, symbol Connector:Screw_Terminal_01x02
- added J13: Thermal 2, Connector_JST:JST_XH_B2B-XH-A_1x02_P2.50mm_Vertical, symbol Connector:Screw_Terminal_01x02
- added J14: CVBS In, Connector_JST:JST_XH_B2B-XH-A_1x02_P2.50mm_Vertical, symbol Connector:Screw_Terminal_01x02
- added J15: CVBS Out, Connector_JST:JST_XH_B2B-XH-A_1x02_P2.50mm_Vertical, symbol Connector:Screw_Terminal_01x02
- added J9: Temp 2, Connector_JST:JST_XH_S3B-XH-A_1x03_P2.50mm_Horizontal, symbol Connector:Screw_Terminal_01x03
- added R1, R2, R3, R4: 365, Resistor_THT:R_Axial_DIN0204_L3.6mm_D1.6mm_P1.90mm_Vertical, symbol Device:R
- added R10, R6, R7, R8, R9: 470, Resistor_THT:R_Axial_DIN0204_L3.6mm_D1.6mm_P1.90mm_Vertical, symbol Device:R
- added Rb0: 4.7k, Resistor_THT:R_Axial_DIN0204_L3.6mm_D1.6mm_P1.90mm_Vertical, symbol Device:R
- added Rp1, Rp2, Rp3, Rp4: 350, Resistor_THT:R_Axial_DIN0204_L3.6mm_D1.6mm_P1.90mm_Vertical, symbol Device:R
- added U1, U2, U3, U4: VOH260A, My Kicad:VOH263A_DIP8, symbol My Kicad Lib:VOH260A
- added U10, U6, U7, U8, U9: 4N35, Package_DIP:DIP-6_W7.62mm, symbol Isolator:4N35
- added U5: LP2950, Package_TO_SOT_THT:TO-92_Inline, symbol Regulator_Linear:LP2950-3.3_TO92
- J1, J2, J3: footprint Connector_Dsub:DSUB-9_Socket_EdgeMount_P2.77mm -> Connector_Dsub:DSUB-9_Pins_Horizontal_P2.77x2.84mm_EdgePinOffset7.70mm_Housed_MountingHolesOffset9.12mm
- J7: footprint (none) -> Connector_JST:JST_XH_S5B-XH-A_1x05_P2.50mm_Horizontal
- J8: value Temp Sensor -> Temp 1; footprint Connector_JST:JST_XH_B3B-XH-A_1x03_P2.50mm_Vertical -> Connector_JST:JST_XH_S3B-XH-A_1x03_P2.50mm_Horizontal
- P1: value Raspberry_Pi_4 -> Pi 5
- Ra0: renamed from R1; footprint Resistor_THT:R_Axial_DIN0204_L3.6mm_D1.6mm_P2.54mm_Vertical -> Resistor_THT:R_Axial_DIN0204_L3.6mm_D1.6mm_P1.90mm_Vertical
- Ra5: renamed from R5; footprint Resistor_THT:R_Axial_DIN0207_L6.3mm_D2.5mm_P7.62mm_Horizontal -> Resistor_THT:R_Axial_DIN0204_L3.6mm_D1.6mm_P1.90mm_Vertical
- Rc5: renamed from R6; footprint Resistor_THT:R_Axial_DIN0207_L6.3mm_D2.5mm_P7.62mm_Horizontal -> Resistor_THT:R_Axial_DIN0204_L3.6mm_D1.6mm_P1.90mm_Vertical
Connections:
- net +3.3V: now also C2.1, C4.1, J9.3 (Pin_3), R2.1, R4.1, Rb0.1, Rp2.1, Rp4.1, U1.8 (VCC), U3.8 (VCC)
- net GND: now also C2.2, C4.2, J9.1 (Pin_1), U1.5 (GND), U10.4, U3.5 (GND), U6.4, U7.4, U8.4, U9.4; no longer J2.9, J7.2 (Pin_2)
- net PTT: no longer P1.13 (GPIO27/SDIO_DAT3)
- net VIDEO: now also J12.1 (Pin_1), J13.1 (Pin_1)
- net GARMIN_IO23: now reaches J2.2
- net GARMIN_IO23: now also U7.2
- net GARMIN_IO25: now reaches J2.3
- net GARMIN_IO25: now also U9.2
- net GARMIN_IO22: now reaches J2.6
- net GARMIN_IO22: now also U6.2
- net GARMIN_IO24: now reaches J2.7
- net GARMIN_IO24: now also U8.2
- net IO22: now reaches P1.15 (GPIO22/SDIO_CLK)
- net IO22: now also U6.5
- net IO23: now reaches P1.16 (GPIO23/SDIO_CMD)
- net IO23: now also U7.5
- net IO24: now reaches P1.18 (GPIO24/SDIO_DAT0)
- net IO24: now also U8.5
- net IO21: now reaches P1.40 (GPIO21/SPI1_SCLK/PCM_DOUT)
- net IO21: now also U10.5
- net GARMIN_SERIAL_RX renamed GARMIN_G3X_RX
- net GARMIN_G3X_RX: now also Rp3.2, U4.6 (VO); no longer P1.8 (GPIO14/UART_TXD)
- net GARMIN_SERIAL_TX renamed GARMIN_G3X_TX
- net GARMIN_G3X_TX: now also U3.3 (CATHODE); no longer P1.10 (GPIO15/UART_RXD)
- net MASTER renamed +12V
- net +12V: now also C5.1, R10.1, R6.1, R7.1, R8.1, R9.1, U5.3 (VI)
- net PAUSE renamed GARMIN_IO21
- net GARMIN_IO21: now also U10.2; no longer P1.37 (GPIO26/SDIO_DAT2)
- net TEMP renamed TEMP1
- net TEMP1: now also P1.37 (GPIO26/SDIO_DAT2); no longer P1.22 (GPIO25/SDIO_DAT1)
- net VIDEO_SERIAL_RX renamed VIDEO_CAM_RX
- net VIDEO_CAM_RX: now also Rp1.2, U2.6 (VO); no longer P1.32 (GPIO12/PWM0)
- net VIDEO_SERIAL_TX renamed VIDEO_CAM_TX
- net VIDEO_CAM_TX: now also U1.3 (CATHODE); no longer P1.33 (GPIO13/PWM1)
- new net: J14.1 (Pin_1), J15.1 (Pin_1)
- new net: J14.2 (Pin_2), J15.2 (Pin_2)
- new net: R7.2, U7.1
- new net: R3.2, U3.2 (ANODE)
- new net: R4.2, U4.2 (ANODE)
- new net: R1.2, U1.2 (ANODE)
- new net: R9.2, U9.1
- new net: R2.2, U2.2 (ANODE)
- new net: R6.2, U6.1
- new net: R8.2, U8.1
- new net: R10.2, U10.1
- new net GARMIN_PI_RX: P1.10 (GPIO15/UART_RXD), Rp4.2, U3.6 (VO)
- new net GARMIN_PI_TX: P1.8 (GPIO14/UART_TXD), U4.3 (CATHODE)
- new net GNDPWR: C1.1, C3.1, C5.2, C6.2, J10.2 (Pin_2), J12.2 (Pin_2), J13.2 (Pin_2), J2.9, J7.2 (Pin_2), U2.5 (GND), U4.5 (GND), U5.2 (GND)
- new net IO25: P1.22 (GPIO25/SDIO_DAT1), U9.5
- new net TEMP2: J9.2 (Pin_2), P1.13 (GPIO27/SDIO_DAT3), Rb0.2
- new net VCC: C1.2, C3.2, C6.1, J10.1 (Pin_1), R1.1, R3.1, Rp1.1, Rp3.1, U2.8 (VCC), U4.8 (VCC), U5.1 (VO)
- new net VIDEO_PI_RX: P1.33 (GPIO13/PWM1/UART4_RXD), Rp2.2, U1.6 (VO)
- new net VIDEO_PI_TX: P1.32 (GPIO12/PWM0/UART4_TXT), U2.3 (CATHODE)
- no-connect marks 10 -> 32
Other:
- moved on the sheet: J1, J2, J3, J4, J5, J6, J7, J8, P1, Ra0, Ra5, Rc5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
