File: hardware/panel/panel.kicad_pcb (KiCad board)
At the start: 2 copper layers, 155 x 40 mm, 30 parts, among them J1 DE9_Socket, U1 Dual Encoder, U2 MCP23017x-x-SP, U3 256x64 OLED, U4 BME280, U5 VEML6030

Commit message: panel and avionics boards
Parts:
- removed C5, C6, C7: 100nf, Capacitor_THT:C_Disc_D5.0mm_W2.5mm_P5.00mm
- removed REF** (x2): MountingHole_3.2mm_M3, MountingHole:MountingHole_3.2mm_M3
- removed U4: BME280, Package_LGA:Bosch_LGA-8_2.5x2.5mm_P0.65mm_ClockwisePinNumbering
- removed U5: VEML6030, My Kicad:VISHAY_VEML6030_2X2X0.87
- added J2: BME280 Board, My Kicad:BME280 Board, F.Cu at (30.0, 21.3)
- added J3: VEML7700 Board, My Kicad:VEML7700 Board, F.Cu at (147.0, 25.4)
- added MH1: MountingHole_3.2mm_M3, MountingHole:MountingHole_3.2mm_M3, F.Cu at (18.5, 18.5)
- added MH2: MountingHole_3.2mm_M3, MountingHole:MountingHole_3.2mm_M3, F.Cu at (18.5, 51.4)
- added MH3: MountingHole_3.2mm_M3, MountingHole:MountingHole_3.2mm_M3, F.Cu at (166.5, 18.5)
- added MH4: MountingHole_3.2mm_M3, MountingHole:MountingHole_3.2mm_M3, F.Cu at (166.5, 51.4)
- D1: value LED -> Red; footprint LED_THT:LED_D5.0mm -> LED_THT:LED_D3.0mm
- D2: value LED -> White; footprint LED_THT:LED_D5.0mm -> LED_THT:LED_D3.0mm
- D3: value LED -> Blue; footprint LED_THT:LED_D5.0mm -> LED_THT:LED_D3.0mm
- D4: value LED -> Yellow; footprint LED_THT:LED_D5.0mm -> LED_THT:LED_D3.0mm
- R8, R9: value 75 -> 39
- U2: value MCP23017x-x-SP -> MCP23017
- moved D1 17.3 mm to (20.8, 31.0)
- moved D4 15.0 mm to (36.8, 31.0)
- moved D2 10.9 mm to (26.2, 31.0)
- moved D3 9.73 mm to (31.5, 31.0)
- moved U1 6.18 mm to (152.5, 51.5)
- moved S1 5.10 mm to (30.0, 44.3)
Connections:
- U3 pad 15: RESET -> unconnected-(U3-RES#-Pad15)
Routing:
- net SDA: track 189.5 -> 144.7 mm, vias 0 -> 1
- net GND: track 44.2 -> 8.19 mm, vias 2 -> 4
- net +3.3V: track 218.1 -> 185.8 mm, vias 1 -> 0
- net Net-(U1-CW_1): track 102.4 -> 128.2 mm, vias 2 -> 1
- net Net-(D1-K): track 15.9 -> 32.7 mm
- net Net-(D1-A): track 98.2 -> 113.0 mm
- net Net-(D2-K): track 16.6 -> 29.9 mm
- net RESET: track 44.2 -> 31.9 mm
- net Net-(U1-CW_2): track 111.5 -> 99.9 mm, vias 2 -> 1
- net Net-(D3-A): track 92.9 -> 103.6 mm
- net SCK: track 175.5 -> 165.8 mm
- net Net-(D3-K): track 16.8 -> 26.1 mm
- net Net-(D2-A): track 98.7 -> 107.7 mm, vias 1 -> 0
- net Net-(U1-W): track 46.5 -> 38.2 mm
- net SCLK: track 83.5 -> 76.4 mm, vias 0 -> 1
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- removed copper zone on B.Cu, net GND
Other:
- board text added: "JLCJLCJLCJLC"
- board text added: "Panel v1"

Commit message: Panel v2
Parts:
- removed R10: 75, Resistor_THT:R_Axial_DIN0207_L6.3mm_D2.5mm_P7.62mm_Horizontal
- removed R9: 39, Resistor_THT:R_Axial_DIN0207_L6.3mm_D2.5mm_P7.62mm_Horizontal
- added C5: 1µf, Capacitor_THT:C_Disc_D5.0mm_W2.5mm_P5.00mm, F.Cu at (88.3, 17.1)
- added SW1: SW_SPST, Button_Switch_THT:SW_PUSH_6mm_H8mm, F.Cu at (21.7, 20.6)
- added SW2: SW_SPST, Button_Switch_THT:SW_PUSH_6mm_H8mm, F.Cu at (31.8, 20.6)
- added SW3: SW_SPST, Button_Switch_THT:SW_PUSH_6mm_H8mm, F.Cu at (21.7, 28.2)
- added SW4: SW_SPST, Button_Switch_THT:SW_PUSH_6mm_H8mm, F.Cu at (31.8, 28.2)
- added U4: LP5816DRLR, My Kicad:LP5816DRLR, B.Cu at (82.0, 19.6)
- J1: moved to F.Cu
- J2: moved to B.Cu
- R7: value 75 -> 4.7k
- R8: value 39 -> 4.7k
- U2: value MCP23017 -> MCP23017x-x-SP
- moved D1 99.4 mm to (119.4, 17.8)
- moved D2 91.6 mm to (116.8, 17.8), turned to 180 degrees
- moved C4 63.1 mm to (123.8, 33.0), turned to 90 degrees
- moved C3 59.1 mm to (120.0, 32.9), turned to 90 degrees
- moved C2 55.6 mm to (116.2, 32.9), turned to 90 degrees
- moved R4 54.0 mm to (123.8, 44.5), turned to 90 degrees
- moved C1 52.5 mm to (112.4, 32.9), turned to 90 degrees
- moved R3 49.0 mm to (120.0, 44.5), turned to 90 degrees
- moved R7 45.6 mm to (97.2, 24.8), turned to 90 degrees
- moved R2 44.3 mm to (116.2, 44.5), turned to 90 degrees
- moved R8 42.7 mm to (93.3, 24.8), turned to 90 degrees
- moved R1 40.0 mm to (112.4, 44.5), turned to 90 degrees
- moved D3 39.4 mm to (68.6, 17.8)
- moved J2 35.1 mm to (62.9, 33.7), turned to 180 degrees
- moved D4 32.1 mm to (66.0, 17.8), turned to 180 degrees
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Connections:
- D1 pad 2: Net-(D1-A) -> +3.3V
- D2 pad 2: Net-(D2-A) -> +3.3V
- D3 pad 2: Net-(D3-A) -> +3.3V
- D4 pad 2: Net-(D4-A) -> +3.3V
- J2 pad 2: +3.3V -> GND
- J2 pad 3: SDA -> SCK
- J2 pad 4: SCK -> SDA
- J2 pad 5: GND -> +3.3V
- J3 pad 1: SDA -> +3.3V
- J3 pad 2: SCK -> unconnected-(J3-Pin_2-Pad2)
- J3 pad 4: unconnected-(J3-Pin_4-Pad4) -> SCK
- J3 pad 5: +3.3V -> SDA
- R7 pad 1: Net-(D1-K) -> SDA
- R7 pad 2: GND -> +3.3V
- R8 pad 1: Net-(D2-K) -> SCK
- R8 pad 2: GND -> +3.3V
- U2 pad 1: Net-(D4-A) -> SW4
- U2 pad 26: Net-(D1-A) -> SW1
- U2 pad 27: Net-(D2-A) -> SW2
- U2 pad 28: Net-(D3-A) -> SW3
- U3 pad 15: unconnected-(U3-RES#-Pad15) -> RESET
Routing:
- net SW3: track 0.00 -> 123.0 mm
- net SW1: track 0.00 -> 122.6 mm, vias 0 -> 2
- net Net-(D1-A): track 113.0 -> 0.00 mm
- net SW2: track 0.00 -> 112.9 mm
- net Net-(D2-A): track 107.7 -> 0.00 mm
- net Net-(D3-A): track 103.6 -> 0.00 mm
- net SW4: track 0.00 -> 103.2 mm
- net Net-(D4-A): track 88.8 -> 0.00 mm
- net Net-(U1-CW_1): track 128.2 -> 46.6 mm, vias 1 -> 0
- net Net-(U1-CW_2): track 99.9 -> 43.8 mm, vias 1 -> 0
- net +3.3V: track 185.8 -> 225.6 mm
- net Net-(U1-CCW_2): track 93.1 -> 53.9 mm
- net Net-(U1-CCW_1): track 103.9 -> 67.2 mm, vias 1 -> 0
- net GND: track 8.19 -> 42.7 mm, vias 4 -> 5
- net SCK: track 165.8 -> 135.1 mm, vias 0 -> 2
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Other:
- outline, holes or cut-outs redrawn
- board text added: "Panel v2"
- board text removed: "Panel v1"
