File: hardware/panel/panel.kicad_sch (KiCad schematic)
At the start: 28 parts, among them J1 DE9_Socket, U1 Dual Encoder, U2 MCP23017x-x-SP, U3 256x64 OLED, U4 BME280, U5 VEML6030

Commit message: panel and avionics boards
Parts:
- removed C5, C6, C7: 100nf, Capacitor_THT:C_Disc_D5.0mm_W2.5mm_P5.00mm, symbol Device:C
- removed U4: BME280, Package_LGA:Bosch_LGA-8_2.5x2.5mm_P0.65mm_ClockwisePinNumbering, symbol Sensor:BME280
- removed U5: VEML6030, My Kicad:VISHAY_VEML6030_2X2X0.87, symbol My Kicad Lib:VEML6030
- added J2: BME280 Board, My Kicad:BME280 Board, symbol Connector:Conn_01x06_Socket
- added J3: VEML7700 Board, My Kicad:VEML7700 Board, symbol Connector:Conn_01x05_Socket
- D1: value LED -> Red; footprint LED_THT:LED_D5.0mm -> LED_THT:LED_D3.0mm
- D2: value LED -> White; footprint LED_THT:LED_D5.0mm -> LED_THT:LED_D3.0mm
- D3: value LED -> Blue; footprint LED_THT:LED_D5.0mm -> LED_THT:LED_D3.0mm
- D4: value LED -> Yellow; footprint LED_THT:LED_D5.0mm -> LED_THT:LED_D3.0mm
- R8, R9: value 75 -> 39
Connections:
- net +3.3V: now also J2.1 (Pin_1), J2.2 (Pin_2), J2.6 (Pin_6), J3.5 (Pin_5)
- net GND: now also J2.5 (Pin_5), J3.3 (Pin_3)
- net RESET: no longer U3.15 (RES#)
- net SCK: now also J2.4 (Pin_4), J3.2 (Pin_2)
- net SDA: now also J2.3 (Pin_3), J3.1 (Pin_1)

Commit message: Panel v2
Parts:
- removed R10: 75, Resistor_THT:R_Axial_DIN0207_L6.3mm_D2.5mm_P7.62mm_Horizontal, symbol Device:R
- removed R9: 39, Resistor_THT:R_Axial_DIN0207_L6.3mm_D2.5mm_P7.62mm_Horizontal, symbol Device:R
- added C5: 1µf, Capacitor_THT:C_Disc_D5.0mm_W2.5mm_P5.00mm, symbol Device:C
- added SW1, SW2, SW3, SW4: SW_SPST, Button_Switch_THT:SW_PUSH_6mm_H8mm, symbol Switch:SW_SPST
- added U4: LP5816DRLR, My Kicad:LP5816DRLR, symbol My Kicad Lib:LP5816DRLR
- R7: value 75 -> 4.7k
- R8: value 39 -> 4.7k
Connections:
- net +3.3V: now also D1.2 (A), D2.2 (A), D3.2 (A), D4.2 (A), J2.5 (Pin_5), J3.1 (Pin_1), R7.2, R8.2, C5.1, U4.4 (VCC); no longer J2.2 (Pin_2), J3.5 (Pin_5)
- net GND: now also J2.2 (Pin_2), C5.2, SW1.1 (A), SW2.1 (A), SW3.1 (A), SW4.1 (A), U4.3 (GND); no longer J2.5 (Pin_5), R7.2, R8.2
- net RESET: now also U3.15 (RES#)
- net SCK: now also J2.3 (Pin_3), J3.4 (Pin_4), R8.1, U4.1 (SCL); no longer J2.4 (Pin_4), J3.2 (Pin_2)
- net SDA: now also J2.4 (Pin_4), J3.5 (Pin_5), R7.1, U4.2 (SDA); no longer J2.3 (Pin_3), J3.1 (Pin_1)
- net at D2.1 (K): now also U4.7 (OUT1); no longer R8.1
- net SW2: now reaches U2.27 (GPA6)
- net SW2: now also SW2.2 (B); no longer D2.2 (A)
- net at D4.1 (K): now also U4.5 (OUT3)
- net SW4: now reaches U2.1 (GPB0)
- net SW4: now also SW4.2 (B); no longer D4.2 (A)
- net at D3.1 (K): now also U4.6 (OUT2)
- net SW3: now reaches U2.28 (GPA7)
- net SW3: now also SW3.2 (B); no longer D3.2 (A)
- net SW1: now reaches U2.26 (GPA5)
- net SW1: now also SW1.2 (B); no longer D1.2 (A)
- net at D1.1 (K): now also U4.8 (OUT0); no longer R7.1
